File: hardware/tapeshnik-mecha/foc/foc.kicad_pcb (KiCad board)
At the start: 2 copper layers, 82 x 43.5 mm, 36 parts, among them J1 Conn_01x03, J2 Conn_01x03, J3 Conn_01x02, J4 Conn_01x07, J5 Conn_01x03, J6 Conn_01x03, U1 STSPIN233, U2 INA181A1IDBVR, U3 MT6701, U4 INA181A1IDBVR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

Commit message: adding a lot of mecha-specific stuff
Parts:
- removed U6: MT6701, Package_SO:SOP-8_3.9x4.9mm_P1.27mm
- added C12: 10nF, Capacitor_SMD:C_0402_1005Metric, F.Cu at (161.3, 97.5)
- added C13: 10nF, Capacitor_SMD:C_0402_1005Metric, F.Cu at (136.7, 98.0)
- added R10: 3K3, Resistor_SMD:R_0402_1005Metric, F.Cu at (138.9, 98.7)
- added R11: 3K3, Resistor_SMD:R_0402_1005Metric, F.Cu at (163.5, 97.9)
- added R7: 33K, Resistor_SMD:R_0402_1005Metric, F.Cu at (162.4, 97.9)
- added R8: 33K, Resistor_SMD:R_0402_1005Metric, F.Cu at (137.8, 98.7)
- added R9: 33K, Resistor_SMD:R_0603_1608Metric, F.Cu at (154.0, 94.0)
- added U10: AS5047D, Package_SO:TSSOP-14_4.4x5mm_P0.65mm, B.Cu at (171.2, 100.0)
- C2, C7: footprint Capacitor_SMD:C_0603_1608Metric -> Capacitor_SMD:C_0805_2012Metric
- C4, C5: moved to B.Cu
- R1, R2, R5, R6: value 0.01/1W -> 0.033/1W
- U3: value MT6701 -> AS5047D; footprint Package_SO:SOP-8_3.9x4.9mm_P1.27mm -> Package_SO:TSSOP-14_4.4x5mm_P0.65mm
- moved C4 5.95 mm to (133.4, 100.7), turned to -90 degrees
- moved C2 0.34 mm to (130.8, 107.8)
- moved C7 0.34 mm to (154.8, 103.0)
- moved C5 0.23 mm to (176.1, 100.0), turned to 90 degrees
- turned U3 to 0 degrees
Connections:
- U1 pad 12: +3V3 -> Net-(U1-ENU)
- U1 pad 13: +3V3 -> Net-(U1-EN/FAULT)
- U1 pad 14: +3V3 -> /~{STANDBY}
- U1 pad 16: +3V3 -> Net-(U1-ENU)
- U1 pad 2: +3V3 -> Net-(U1-ENU)
- U3 pad 1: +3V3 -> /~{SSI_CS1}
- U3 pad 2: +3V3 -> /SCK
- U3 pad 3: unconnected-(U3-OUT-Pad3) -> /MISO
- U3 pad 4: GND -> /MOSI
- U3 pad 5: unconnected-(U3-PUSH-Pad5) -> GND
- U3 pad 6: /MISO -> unconnected-(U3-B-Pad6)
- U3 pad 7: /SCK -> unconnected-(U3-A-Pad7)
- U3 pad 8: /~{SSI_CS1} -> unconnected-(U3-W/PWM-Pad8)
- U5 pad 7: unconnected-(U5-GP15-Pad7) -> /~{STANDBY}
- U7 pad 12: +3V3 -> Net-(U7-ENU)
- U7 pad 13: +3V3 -> Net-(U7-EN/FAULT)
- U7 pad 14: +3V3 -> /~{STANDBY}
- U7 pad 16: +3V3 -> Net-(U7-ENU)
- U7 pad 2: +3V3 -> Net-(U7-ENU)
Routing:
- net /~{STANDBY}: track 0.00 -> 70.7 mm, vias 0 -> 3
- net GND: track 165.3 -> 232.6 mm, vias 70 -> 101
- net /MOSI: track 27.2 -> 83.9 mm, vias 0 -> 2
- net Net-(U1-ENU): track 0.00 -> 10.7 mm, vias 0 -> 3
- net Net-(U7-ENU): track 0.00 -> 10.6 mm, vias 0 -> 3
- net +3V3: track 199.4 -> 189.9 mm, vias 15 -> 9
- net /~{SSI_CS2}: track 66.7 -> 61.6 mm, vias 0 -> 2
- net Net-(U7-EN/FAULT): track 0.00 -> 3.92 mm
- net /PWM1_V: track 37.1 -> 40.5 mm
- net Net-(U1-EN/FAULT): track 0.00 -> 3.14 mm
- net /~{SSI_CS1}: track 16.6 -> 14.0 mm
- net /PWM2_V: track 69.9 -> 72.4 mm
- net /SENSEW1: track 70.4 -> 72.6 mm
- net /SENSEV1: track 65.7 -> 67.7 mm
- net /SCK: track 79.8 -> 78.0 mm
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Other:
- board text added: "OPTICAL"
- board text added: "~{STANDBY}"
- board text removed: "~{CS}"
