File: hardware/tapeshnik-mecha/platen-heads-butter/platen-heads-butter.kicad_pcb (KiCad board)
At the start: 2 copper layers, 137.6 x 83 mm, 16 parts

Commit message: adding a lot of mecha-specific stuff
Parts:
- removed the REF** at (232.0, 21.5)
- removed the REF** at (104.0, 21.0)
- added J1: Conn_01x09, Connector_PinHeader_2.54mm:PinHeader_1x09_P2.54mm_Vertical, F.Cu at (190.8, 19.5)
Routing:
- added copper zone on B.Cu, net GND
- added copper zone on F.Cu, net GND
Other:
- outline, holes or cut-outs redrawn
- board text added: "BUTTER"
- board text added: "TAPESHNIK"
- board text added: "svofski 2023 https://caglrc.cc/tapeshnik"
