File: hardware/tapeshnik-mecha/platen-motors/platen-motors.kicad_pcb (KiCad board)
At the start: 2 copper layers, 129 x 80 mm, 25 parts

Commit message: adding a lot of mecha-specific stuff
Parts:
- removed the REF** at (136.0, 98.1)
- removed the REF** at (93.5, 98.1)
- removed the REF** at (158.7, 118.5)
- removed the REF** at (61.8, 68.6)
- removed the REF** at (81.5, 118.4)
- added J1: Conn_01x07, Connector_PinHeader_2.54mm:PinHeader_1x07_P2.54mm_Vertical, F.Cu at (63.0, 120.1)
- added J2: Conn_01x07, Connector_PinHeader_2.54mm:PinHeader_1x07_P2.54mm_Vertical, F.Cu at (63.1, 126.1)
- added J3: Conn_01x03, Connector_PinHeader_2.54mm:PinHeader_1x03_P2.54mm_Vertical, F.Cu at (157.8, 126.1)
- added M1: Motor_Servo, Connector_PinHeader_2.54mm:PinHeader_1x03_P2.54mm_Vertical, F.Cu at (152.7, 92.6)
- added REF**: MountingHole_3.2mm_M3, MountingHole:MountingHole_3.2mm_M3, F.Cu at (89.8, 80.1)
- added REF**: MountingHole_3.2mm_M3, MountingHole:MountingHole_3.2mm_M3, F.Cu at (89.8, 116.6)
- added REF**: MountingHole_3.2mm_M3, MountingHole:MountingHole_3.2mm_M3, F.Cu at (139.8, 80.1)
- added REF**: MountingHole_3.2mm_M3, MountingHole:MountingHole_3.2mm_M3, F.Cu at (139.8, 116.6)
- added U1: ~, MechanicalParts:AS5600-breakout-23x23, F.Cu at (93.5, 98.1)
- added U2: ~, MechanicalParts:AS5600-breakout-23x23, F.Cu at (136.0, 98.1)
- REF** (x2): moved to B.Cu
- turned REF** to 180 degrees (x2)
Routing:
- net +3V3: track 0.00 -> 146.9 mm
- net GND: track 0.00 -> 124.4 mm
- net Net-(J2-Pin_3): track 0.00 -> 84.4 mm, vias 0 -> 1
- net Net-(J2-Pin_4): track 0.00 -> 82.3 mm
- net Net-(J2-Pin_5): track 0.00 -> 76.8 mm
- net Net-(J2-Pin_6): track 0.00 -> 71.4 mm
- net Net-(J2-Pin_7): track 0.00 -> 65.8 mm
- net (no net): track 0.00 -> 61.5 mm
- net Net-(J1-Pin_3): track 0.00 -> 42.7 mm
- net /LIFT_PWR: track 0.00 -> 38.0 mm
- net /LIFT_PWM: track 0.00 -> 36.8 mm
- net Net-(J1-Pin_4): track 0.00 -> 35.9 mm
- net /LIFT_GND: track 0.00 -> 35.8 mm
- net Net-(J1-Pin_5): track 0.00 -> 30.4 mm
- net Net-(J1-Pin_6): track 0.00 -> 26.0 mm
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- added copper zone on B.Cu, net GND
- added copper zone on F.Cu, net GND
Other:
- board text added: "3V3"
- board text added: "DIR"
- board text added: "GND"
- board text added: "GPO"
- board text added: "LIFT"
- board text added: "MOTOR PLATEN"
- board text added: "OUT"
- board text added: "PWM"
- board text added: "PWR"
- board text added: "SCL"
- board text added: "SDA"
- board text added: "TAPESHNIK"
- board text added: "svofski 2023 https://caglrc.cc/tapeshnik"
