File: hardware/tapeshnik-mecha/platen-heads/platen-heads.kicad_pcb (KiCad board)
At the start: 2 copper layers, 137.6 x 83 mm, 27 parts

Commit message: adding a lot of mecha-specific stuff
Parts:
- removed the REF** at (104.0, 21.0)
- removed the REF** at (232.0, 21.5)
- added J1: Conn_01x07, PCB_Edge_Connectors:EDGE-2.54-7x, F.Cu at (142.6, 22.0)
- added J2: Conn_01x07, Connector_JST:JST_SH_SM07B-SRSS-TB_1x07-1MP_P1.00mm_Horizontal, F.Cu at (106.0, 20.2)
- added J3: Conn_01x09, Connector_JST:JST_SH_SM09B-SRSS-TB_1x09-1MP_P1.00mm_Horizontal, F.Cu at (221.8, 20.5)
- added J4: Conn_01x09, Connector_PinHeader_2.54mm:PinHeader_1x09_P2.54mm_Vertical, F.Cu at (190.8, 19.5)
Routing:
- net GND: track 0.00 -> 52.3 mm
- net Net-(J1-Pin_1): track 0.00 -> 45.1 mm
- net Net-(J1-Pin_3): track 0.00 -> 42.8 mm
- net Net-(J3-Pin_1): track 0.00 -> 41.4 mm, vias 0 -> 1
- net Net-(J1-Pin_4): track 0.00 -> 41.3 mm
- net Net-(J1-Pin_5): track 0.00 -> 39.7 mm
- net Net-(J1-Pin_6): track 0.00 -> 38.2 mm
- net Net-(J3-Pin_2): track 0.00 -> 38.0 mm
- net Net-(J1-Pin_7): track 0.00 -> 34.3 mm
- net Net-(J3-Pin_3): track 0.00 -> 33.1 mm, vias 0 -> 1
- net Net-(J3-Pin_4): track 0.00 -> 30.0 mm
- net Net-(J3-Pin_5): track 0.00 -> 25.3 mm, vias 0 -> 1
- net Net-(J3-Pin_6): track 0.00 -> 21.6 mm
- net Net-(J3-Pin_7): track 0.00 -> 17.1 mm, vias 0 -> 1
- net Net-(J3-Pin_8): track 0.00 -> 12.6 mm
- added copper zone on B.Cu, net GND
- added copper zone on F.Cu, net GND
Other:
- board text added: "TAPESHNIK"
- board text added: "TOP PLATEN"
- board text added: "svofski 2023 https://caglrc.cc/tapeshnik"

Commit message: kicad file updates
Parts:
- added REF**: MountingHole_3.2mm_M3, MountingHole:MountingHole_3.2mm_M3, F.Cu at (107.9, 83.2)
Changed lines of the file:
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@@
+    (pad "" np_thru_hole circle (at 0 0) (size 3.2 3.2) (drill 3.2) (layers "*.Cu" "*.Mask"))
+  )
+  (footprint "MountingHole:MountingHole_3.2mm_M3" (layer "F.Cu")
+    (at 107.88 83.18)
+    (descr "Mounting Hole 3.2mm, no annular, M3")
+    (tags "mounting hole 3.2mm no annular m3")
+    (attr exclude_from_pos_files exclude_from_bom)
+    (fp_text reference "REF**" (at 0 -4.2) (layer "F.SilkS") hide
+        (effects (font (size 1 1) (thickness 0.15)))
+    )
+    (fp_text value "MountingHole_3.2mm_M3" (at 0 4.2) (layer "F.Fab") hide
+        (effects (font (size 1 1) (thickness 0.15)))
+    )
+    (fp_text user "${REFERENCE}" (at 0 0) (layer "F.Fab")
+        (effects (font (size 1 1) (thickness 0.15)))
+    )
+    (fp_circle (center 0 0) (end 3.2 0)
+      (stroke (width 0.15) (type solid)) (fill none) (layer "Cmts.User"))
+    (fp_circle (center 0 0) (end 3.45 0)
+      (stroke (width 0.05) (type solid)) (fill none) (layer "F.CrtYd"))
     (pad "" np_thru_hole circle (at 0 0) (size 3.2 3.2) (drill 3.2) (layers "*.Cu" "*.Mask"))
   )
@@
   (gr_arc (start 130.5 33) (mid 130.146447 32.853553) (end 130 32.5)
     (stroke (width 0.1) (type default)) (layer "Edge.Cuts"))
-  (gr_text "svofski 2023 https://caglrc.cc/tapeshnik" (at 135.4 49.4) (layer "Edge.Cuts")
+  (gr_text "svofski 2023 https://caglrc.cc/tapeshnik" (at 135.4 49.4) (layer "F.SilkS")
     (effects (font (size 1 0.8) (thickness 0.15)) (justify left bottom))
   )
-  (gr_text "TOP PLATEN" (at 148.4 47.1) (layer "Edge.Cuts")
+  (gr_text "TOP PLATEN" (at 148.4 47.1) (layer "F.SilkS")
     (effects (font (size 1.5 1.5) (thickness 0.2)) (justify left bottom))
   )
-  (gr_text "TAPESHNIK" (at 135.4 47.1) (layer "Edge.Cuts" knockout)
+  (gr_text "TAPESHNIK" (at 135.4 47.1) (layer "F.SilkS" knockout)
     (effects (font (size 1.5 1.5) (thickness 0.375) bold) (justify left bottom))
   )
