File: hardware/tapeshnik-mecha/pwm3389_pcb_edge/pwm3389_pcb_edge.kicad_sch (KiCad schematic)
At the start: 15 parts, among them J2 Conn_01x07, U1 PMW3360DM-T2QU, U2 TPS73601DBV

Commit message: updates kicad files + doc
Other:
- note added: "LDO can be replaced by SPX3819M5-1.8V: - R4, R5 don't install"
